Commit message: feat: unify colored URDF via per-material split STL + top-level materials
- Replace DAE-baked arm colors with 23 per-material STL visuals referencing
  top-level <material> rgba extracted from DAE diffuse colors
  (extract_dae_colors.py) and regenerated by unify_arm_urdf.py
- Sync colors across URDF, MuJoCo MJCF and web simulator; drop
  REAL_FINISH_GROUPS face-index hack in rebot-sim.js, use URDF material
  names + URDF_FINISH_PARAMS gloss table instead
- Add standalone shareable description/ package (URDF with relative mesh
  paths + 44 STLs + README) usable by URDFLoader/RViz/MuJoCo directly
- Server switches to reBot-DevArm_colored.urdf
- Final palette: anodized_grey = CNC matte silver-grey 0.62 0.63 0.61

File: description/reBot-DevArm_colored.urdf (robot description, URDF)
Before this commit: robot reBot-DevArm_colored, 10 links, 9 joints
Links:
- link base_link: geometry collision mesh filename=meshes/base_link.STL; visual mesh filename=meshes/colored_base_link_hardware_black.stl
- link end_link: geometry collision mesh filename=meshes/gripper_base.stl; visual mesh filename=meshes/colored_gripper_base_hardware_black.stl
- link finger_left_link: geometry collision mesh filename=meshes/left_finger.stl; visual mesh filename=meshes/colored_left_finger_carriage_grey.stl
- link finger_right_link: geometry collision mesh filename=meshes/right_finger.stl; visual mesh filename=meshes/colored_right_finger_carriage_grey.stl
- link link1: geometry collision mesh filename=meshes/link1.STL; visual mesh filename=meshes/colored_link1_anodized_grey.stl
- link link2: geometry collision mesh filename=meshes/link2.STL; visual mesh filename=meshes/colored_link2_anodized_grey.stl
- link link3: geometry collision mesh filename=meshes/link3.STL; visual mesh filename=meshes/colored_link3_anodized_grey.stl
- link link4: geometry collision mesh filename=meshes/link4.STL; visual mesh filename=meshes/colored_link4_anodized_grey.stl
- link link5: geometry collision mesh filename=meshes/link5.STL; visual mesh filename=meshes/colored_link5_anodized_grey.stl
- link link6: geometry collision mesh filename=meshes/link6.STL; visual mesh filename=meshes/colored_link6_hardware_black.stl
