Commit message: fix(sim): prevent magnetic snap when MuJoCo physics active + widen gripper to 100mm
Physics-snap fix:
- Add mujocoPhysicsActive flag so updateCarriedObject/attachObject bail
  out whenever live physics feedback is streaming, not only after the
  first object_states message arrives
- applyMujocoObjectStates marks ownership unconditionally on any
  object_states message, closing the startup timing window
- rebot-ros-ui propagates physics-active state from joint_states and
  syncs it every second in updateDiagnostics; attachSimCarriedObject
  skips fake attach when physics is running

Gripper travel widened to 100mm total across URDF/MuJoCo XML/configs.

Cache-bust to v80-physics-active-snapfix so the PWA picks up the change.

File: reBotArm_ros2_DM/src/rebotarm_bringup/description/urdf/ReBot_Arm_DM.urdf (robot description, URDF)
Before this commit: robot ReBot_Arm_DM, 10 links, 9 joints
Joints:
- joint finger_left: limit lower=0 upper=0.0285 effort=8 velocity=0.08 -> lower=0 upper=0.05 effort=8 velocity=0.08
- joint finger_right: limit lower=-0.0285 upper=0 effort=8 velocity=0.08 -> lower=-0.05 upper=0 effort=8 velocity=0.08

File: reBotArm_ros2_DM/src/rebotarm_moveit_config/config/rebotarm.ros2_control.xacro (robot description, xacro)
@@ -61,8 +61,8 @@
         </state_interface>
       </joint>
-      <joint name="gripper_joint1">
+      <joint name="finger_left">
         <command_interface name="position"/>
         <state_interface name="position">
-          <param name="initial_value">${initial_positions['gripper_joint1']}</param>
+          <param name="initial_value">${initial_positions['finger_left']}</param>
         </state_interface>
         <state_interface name="velocity">
@@ -70,8 +70,7 @@
         </state_interface>
       </joint>
-      <joint name="gripper_joint2">
-        <command_interface name="position"/>
+      <joint name="finger_right">
         <state_interface name="position">
-          <param name="initial_value">${initial_positions['gripper_joint2']}</param>
+          <param name="initial_value">${initial_positions['finger_right']}</param>
         </state_interface>
         <state_interface name="velocity">

File: reBotArm_ros2_DM/src/rebotarm_moveit_config/config/rebotarm.urdf.xacro (robot description, xacro)
@@ -1,11 +1,11 @@
 <?xml version="1.0"?>
-<robot xmlns:xacro="http://www.ros.org/wiki/xacro" name="reBot_B601_DM_with_gripper">
+<robot xmlns:xacro="http://www.ros.org/wiki/xacro" name="ReBot_Arm_DM">
   <xacro:arg name="initial_positions_file" default="$(find rebotarm_moveit_config)/config/initial_positions.yaml"/>
-  <xacro:include filename="$(find rebotarm_bringup)/description/urdf/reBot_B601_DM_with_gripper.urdf"/>
+  <xacro:include filename="$(find rebotarm_bringup)/description/urdf/ReBot_Arm_DM.urdf"/>
   <xacro:include filename="$(find rebotarm_moveit_config)/config/rebotarm.ros2_control.xacro"/>
   <link name="gripper_tcp"/>
   <joint name="gripper_tcp_joint" type="fixed">
-    <origin xyz="-0.0443 0 0" rpy="0 0 0"/>
-    <parent link="gripper_link"/>
+    <origin xyz="-0.105 0 0" rpy="0 0 0"/>
+    <parent link="end_link"/>
     <child link="gripper_tcp"/>
   </joint>
